File: misc.sch (KiCad schematic (older format))
At the start: 10 parts, among them J11 USB_OTG, U3 RT9193-28, U4 AP7313-30SAG

Commit message: Changed the package of R, C and L to 1206 for hand soldering.
Parts:
- C35: footprint Capacitors_THT:CP_Radial_D5.0mm_P2.50mm -> Capacitor_THT:CP_Radial_D5.0mm_P2.50mm
- C36, C37, C38: footprint Capacitors_SMD:C_0805 -> Capacitor_SMD:C_1206_3216Metric_Pad1.33x1.80mm_HandSolder
- C40: footprint Capacitors_SMD:C_0603 -> Capacitor_SMD:C_1206_3216Metric_Pad1.33x1.80mm_HandSolder
- D1, D2, U4: footprint TO_SOT_Packages_SMD:SOT-23 -> Package_TO_SOT_SMD:SOT-23
- J11: footprint Connectors:USB_Mini-B -> Connector_USB:USB_Micro-B_Wuerth_629105150521
- U3: footprint TO_SOT_Packages_SMD:SOT-23-5 -> Package_TO_SOT_SMD:SOT-23-5
Changed lines of the file:
@@
 F 0 "C38" H 7175 3100 50  0000 L CNN
 F 1 "10uF" H 7175 2900 50  0000 L CNN
-F 2 "Capacitors_SMD:C_0805" H 7188 2850 50  0001 C CNN
+F 2 "Capacitor_SMD:C_1206_3216Metric_Pad1.33x1.80mm_HandSolder" H 7188 2850 50  0001 C CNN
 F 3 "" H 7150 3000 50  0001 C CNN
 	1    7150 3000
@@
 F 0 "C37" H 6475 3050 50  0000 L CNN
 F 1 "10uF" H 6475 2850 50  0000 L CNN
-F 2 "Capacitors_SMD:C_0805" H 6488 2800 50  0001 C CNN
+F 2 "Capacitor_SMD:C_1206_3216Metric_Pad1.33x1.80mm_HandSolder" H 6488 2800 50  0001 C CNN
 F 3 "" H 6450 2950 50  0001 C CNN
 	1    6450 2950
@@
 F 0 "C36" H 5375 2000 50  0000 L CNN
 F 1 "10uF" H 5375 1800 50  0000 L CNN
-F 2 "Capacitors_SMD:C_0805" H 5388 1750 50  0001 C CNN
+F 2 "Capacitor_SMD:C_1206_3216Metric_Pad1.33x1.80mm_HandSolder" H 5388 1750 50  0001 C CNN
 F 3 "" H 5350 1900 50  0001 C CNN
 	1    5350 1900
@@
 F 0 "J11" H 7600 4150 50  0000 L CNN
 F 1 "USB_OTG" H 7600 4050 50  0000 L CNN
-F 2 "Connectors:USB_Mini-B" H 7950 3650 50  0001 C CNN
+F 2 "Connector_USB:USB_Micro-B_Wuerth_629105150521" H 7950 3650 50  0001 C CNN
 F 3 "" H 7950 3650 50  0001 C CNN
 	1    7800 3700
@@
 F 0 "C35" H 4625 3050 50  0000 L CNN
 F 1 "100uF" H 4625 2850 50  0000 L CNN
-F 2 "Capacitors_THT:CP_Radial_D5.0mm_P2.50mm" H 4638 2800 50  0001 C CNN
+F 2 "Capacitor_THT:CP_Radial_D5.0mm_P2.50mm" H 4638 2800 50  0001 C CNN
 F 3 "" H 4600 2950 50  0001 C CNN
 	1    4600 2950
@@
 F 0 "U4" H 6650 2675 50  0000 C CNN
 F 1 "AP7313-30SAG" H 6400 2750 50  0000 L CNN
-F 2 "TO_SOT_Packages_SMD:SOT-23" H 6800 2775 50  0001 C CIN
+F 2 "Package_TO_SOT_SMD:SOT-23" H 6800 2775 50  0001 C CIN
 F 3 "" H 6800 2500 50  0001 C CNN
 	1    6800 2550
@@
 F 0 "U3" H 5900 1875 50  0000 C CNN
 F 1 "RT9193-28" H 6075 1875 50  0000 L CNN
-F 2 "TO_SOT_Packages_SMD:SOT-23-5" H 6150 1975 50  0001 C CIN
+F 2 "Package_TO_SOT_SMD:SOT-23-5" H 6150 1975 50  0001 C CIN
 F 3 "" H 6150 1750 50  0001 C CNN
 	1    6150 1650
@@
 F 0 "C40" H 5725 2100 50  0000 L CNN
 F 1 "22nF" H 5725 1900 50  0000 L CNN
-F 2 "Capacitors_SMD:C_0603" H 5738 1850 50  0001 C CNN
+F 2 "Capacitor_SMD:C_1206_3216Metric_Pad1.33x1.80mm_HandSolder" H 5738 1850 50  0001 C CNN
 F 3 "" H 5700 2000 50  0001 C CNN
 	1    5700 2000
@@
 F 0 "D1" H 4900 3500 50  0000 C CNN
 F 1 "BAV99LT1G" H 4850 3700 50  0000 C CNN
-F 2 "TO_SOT_Packages_SMD:SOT-23" H 4850 3600 50  0001 C CNN
+F 2 "Package_TO_SOT_SMD:SOT-23" H 4850 3600 50  0001 C CNN
 F 3 "" H 4850 3600 50  0001 C CNN
 	1    4850 3600
@@
 F 0 "D2" H 5250 3500 50  0000 C CNN
 F 1 "BAV99LT1G" H 5200 3700 50  0000 C CNN
-F 2 "TO_SOT_Packages_SMD:SOT-23" H 5200 3600 50  0001 C CNN
+F 2 "Package_TO_SOT_SMD:SOT-23" H 5200 3600 50  0001 C CNN
 F 3 "" H 5200 3600 50  0001 C CNN
 	1    5200 3600
@@
 $EndComp
 Wire Wire Line
-	4600 2650 6250 2650
+	4600 2650 4950 2650
 Connection ~ 5100 2650
 Wire Wire Line
-	4200 3700 7500 3700
-Wire Wire Line
-	4200 3800 7500 3800
+	4200 3700 4500 3700
+Wire Wire Line
+	4200 3800 5000 3800
 Wire Wire Line
 	5200 4000 5200 3900
@@
 	6450 2800 6450 2550
 Wire Wire Line
-	6250 2550 6500 2550
-Wire Wire Line
-	7100 2550 7450 2550
+	6250 2550 6450 2550
+Wire Wire Line
+	7100 2550 7150 2550
 Wire Wire Line
 	7150 2550 7150 2850
@@
 Connection ~ 6450 2550
 Wire Wire Line
-	7450 1550 7450 3500
+	7450 1550 7450 2550
 Connection ~ 7150 2550
 Wire Wire Line
@@
 	5500 1550 5500 1500
 Wire Wire Line
-	5500 1500 5150 1500
+	5500 1500 5350 1500
 Wire Wire Line
 	7150 1850 7000 1850
@@
 	5000 3600 5000 3800
 Connection ~ 5000 3800
+Wire Wire Line
+	5100 2650 5200 2650
+Wire Wire Line
+	5200 2650 6250 2650
+Wire Wire Line
+	6450 2550 6500 2550
+Wire Wire Line
+	7150 2550 7450 2550
+Wire Wire Line
+	5350 1500 5150 1500
+Wire Wire Line
+	7450 2550 7450 3500
+Wire Wire Line
+	4950 2650 5100 2650
+Wire Wire Line
+	4500 3700 7500 3700
+Wire Wire Line
+	5000 3800 7500 3800
 $EndSCHEMATC
