File: msi001.sch (KiCad schematic (older format))
At the start: 19 parts, among them U2 msi001

Commit message: Changed the package of R, C and L to 1206 for hand soldering.
Parts:
- C11, C12, C13, C14, C15, C16, C17, C19, C20, C21, C22, C23, C24, C25, C26: footprint Capacitors_SMD:C_0603 -> Capacitor_SMD:C_1206_3216Metric_Pad1.33x1.80mm_HandSolder
- C18: footprint Capacitors_SMD:C_0805 -> Capacitor_SMD:C_1206_3216Metric_Pad1.33x1.80mm_HandSolder
- C43: footprint Capacitor_SMD:C_0603_1608Metric_Pad1.08x0.95mm_HandSolder -> Capacitor_SMD:C_1206_3216Metric_Pad1.33x1.80mm_HandSolder
- R2: footprint Resistors_SMD:R_0603 -> Resistor_SMD:R_1206_3216Metric_Pad1.30x1.75mm_HandSolder
- U2: footprint Housings_DFN_QFN:QFN-40-1EP_6x6mm_Pitch0.5mm -> Package_DFN_QFN:QFN-40-1EP_6x6mm_P0.5mm_EP4.6x4.6mm_ThermalVias
Changed lines of the file:
@@
 F 0 "C11" H 3675 3200 50  0000 L CNN
 F 1 "10nF" H 3675 3000 50  0000 L CNN
-F 2 "Capacitors_SMD:C_0603" H 3688 2950 50  0001 C CNN
+F 2 "Capacitor_SMD:C_1206_3216Metric_Pad1.33x1.80mm_HandSolder" H 3688 2950 50  0001 C CNN
 F 3 "" H 3650 3100 50  0001 C CNN
 	1    3650 3100
@@
 F 0 "C16" H 4825 2550 50  0000 L CNN
 F 1 "100nF" H 4825 2350 50  0000 L CNN
-F 2 "Capacitors_SMD:C_0603" H 4838 2300 50  0001 C CNN
+F 2 "Capacitor_SMD:C_1206_3216Metric_Pad1.33x1.80mm_HandSolder" H 4838 2300 50  0001 C CNN
 F 3 "" H 4800 2450 50  0001 C CNN
 	1    4800 2450
@@
 F 0 "C17" H 5025 2350 50  0000 L CNN
 F 1 "100nF" H 5025 2150 50  0000 L CNN
-F 2 "Capacitors_SMD:C_0603" H 5038 2100 50  0001 C CNN
+F 2 "Capacitor_SMD:C_1206_3216Metric_Pad1.33x1.80mm_HandSolder" H 5038 2100 50  0001 C CNN
 F 3 "" H 5000 2250 50  0001 C CNN
 	1    5000 2250
@@
 F 0 "C18" H 5375 2000 50  0000 L CNN
 F 1 "1uF" H 5375 1800 50  0000 L CNN
-F 2 "Capacitors_SMD:C_0805" H 5388 1750 50  0001 C CNN
+F 2 "Capacitor_SMD:C_1206_3216Metric_Pad1.33x1.80mm_HandSolder" H 5388 1750 50  0001 C CNN
 F 3 "" H 5350 1900 50  0001 C CNN
 	1    5350 1900
@@
 F 0 "C20" H 5925 2000 50  0000 L CNN
 F 1 "10nF" H 5925 1800 50  0000 L CNN
-F 2 "Capacitors_SMD:C_0603" H 5938 1750 50  0001 C CNN
+F 2 "Capacitor_SMD:C_1206_3216Metric_Pad1.33x1.80mm_HandSolder" H 5938 1750 50  0001 C CNN
 F 3 "" H 5900 1900 50  0001 C CNN
 	1    5900 1900
@@
 F 0 "C21" H 6275 2000 50  0000 L CNN
 F 1 "10nF" H 6275 1800 50  0000 L CNN
-F 2 "Capacitors_SMD:C_0603" H 6288 1750 50  0001 C CNN
+F 2 "Capacitor_SMD:C_1206_3216Metric_Pad1.33x1.80mm_HandSolder" H 6288 1750 50  0001 C CNN
 F 3 "" H 6250 1900 50  0001 C CNN
 	1    6250 1900
@@
 F 0 "C24" H 7275 2900 50  0000 L CNN
 F 1 "10nF" H 7275 2700 50  0000 L CNN
-F 2 "Capacitors_SMD:C_0603" H 7288 2650 50  0001 C CNN
+F 2 "Capacitor_SMD:C_1206_3216Metric_Pad1.33x1.80mm_HandSolder" H 7288 2650 50  0001 C CNN
 F 3 "" H 7250 2800 50  0001 C CNN
 	1    7250 2800
@@
 F 0 "C22" H 7075 3300 50  0000 L CNN
 F 1 "6800pF" V 7100 2850 50  0000 L CNN
-F 2 "Capacitors_SMD:C_0603" H 7088 3050 50  0001 C CNN
+F 2 "Capacitor_SMD:C_1206_3216Metric_Pad1.33x1.80mm_HandSolder" H 7088 3050 50  0001 C CNN
 F 3 "" H 7050 3200 50  0001 C CNN
 	1    7050 3200
@@
 F 0 "C23" H 7075 3600 50  0000 L CNN
 F 1 "33nF" V 7100 3150 50  0000 L CNN
-F 2 "Capacitors_SMD:C_0603" H 7088 3350 50  0001 C CNN
+F 2 "Capacitor_SMD:C_1206_3216Metric_Pad1.33x1.80mm_HandSolder" H 7088 3350 50  0001 C CNN
 F 3 "" H 7050 3500 50  0001 C CNN
 	1    7050 3500
@@
 F 0 "C26" H 8075 3400 50  0000 L CNN
 F 1 "10nF" H 8075 3200 50  0000 L CNN
-F 2 "Capacitors_SMD:C_0603" H 8088 3150 50  0001 C CNN
+F 2 "Capacitor_SMD:C_1206_3216Metric_Pad1.33x1.80mm_HandSolder" H 8088 3150 50  0001 C CNN
 F 3 "" H 8050 3300 50  0001 C CNN
 	1    8050 3300
@@
 F 0 "R2" V 7730 3350 50  0000 C CNN
 F 1 "390R" V 7650 3350 50  0000 C CNN
-F 2 "Resistors_SMD:R_0603" V 7580 3350 50  0001 C CNN
+F 2 "Resistor_SMD:R_1206_3216Metric_Pad1.30x1.75mm_HandSolder" V 7580 3350 50  0001 C CNN
 F 3 "" H 7650 3350 50  0001 C CNN
 	1    7650 3350
@@
 F 0 "C19" H 5625 4900 50  0000 L CNN
 F 1 "10nF" H 5625 4700 50  0000 L CNN
-F 2 "Capacitors_SMD:C_0603" H 5638 4650 50  0001 C CNN
+F 2 "Capacitor_SMD:C_1206_3216Metric_Pad1.33x1.80mm_HandSolder" H 5638 4650 50  0001 C CNN
 F 3 "" H 5600 4800 50  0001 C CNN
 	1    5600 4800
@@
 F 0 "C12" H 3675 3900 50  0000 L CNN
 F 1 "10nF" H 3675 3700 50  0000 L CNN
-F 2 "Capacitors_SMD:C_0603" H 3688 3650 50  0001 C CNN
+F 2 "Capacitor_SMD:C_1206_3216Metric_Pad1.33x1.80mm_HandSolder" H 3688 3650 50  0001 C CNN
 F 3 "" H 3650 3800 50  0001 C CNN
 	1    3650 3800
@@
 F 0 "C13" H 3975 4350 50  0000 L CNN
 F 1 "10nF" H 3975 4150 50  0000 L CNN
-F 2 "Capacitors_SMD:C_0603" H 3988 4100 50  0001 C CNN
+F 2 "Capacitor_SMD:C_1206_3216Metric_Pad1.33x1.80mm_HandSolder" H 3988 4100 50  0001 C CNN
 F 3 "" H 3950 4250 50  0001 C CNN
 	1    3950 4250
@@
 F 0 "C14" H 4275 4500 50  0000 L CNN
 F 1 "10nF" H 4275 4300 50  0000 L CNN
-F 2 "Capacitors_SMD:C_0603" H 4288 4250 50  0001 C CNN
+F 2 "Capacitor_SMD:C_1206_3216Metric_Pad1.33x1.80mm_HandSolder" H 4288 4250 50  0001 C CNN
 F 3 "" H 4250 4400 50  0001 C CNN
 	1    4250 4400
@@
 F 0 "C15" H 4575 4700 50  0000 L CNN
 F 1 "10nF" H 4575 4500 50  0000 L CNN
-F 2 "Capacitors_SMD:C_0603" H 4588 4450 50  0001 C CNN
+F 2 "Capacitor_SMD:C_1206_3216Metric_Pad1.33x1.80mm_HandSolder" H 4588 4450 50  0001 C CNN
 F 3 "" H 4550 4600 50  0001 C CNN
 	1    4550 4600
@@
 F 0 "U2" H 4900 3000 39  0000 C CNN
 F 1 "msi001" H 5450 2550 39  0000 C CNN
-F 2 "Housings_DFN_QFN:QFN-40-1EP_6x6mm_Pitch0.5mm" H 4900 3000 39  0001 C CNN
+F 2 "Package_DFN_QFN:QFN-40-1EP_6x6mm_P0.5mm_EP4.6x4.6mm_ThermalVias" H 4900 3000 39  0001 C CNN
 F 3 "" H 4900 3000 39  0001 C CNN
 	1    4900 3000
@@
 F 0 "C25" H 7775 4100 50  0000 L CNN
 F 1 "10nF" H 7775 3900 50  0000 L CNN
-F 2 "Capacitors_SMD:C_0603" H 7788 3850 50  0001 C CNN
+F 2 "Capacitor_SMD:C_1206_3216Metric_Pad1.33x1.80mm_HandSolder" H 7788 3850 50  0001 C CNN
 F 3 "" H 7750 4000 50  0001 C CNN
 	1    7750 4000
@@
 F 0 "C43" H 6725 4400 50  0000 L CNN
 F 1 "10nF" H 6725 4200 50  0000 L CNN
-F 2 "Capacitor_SMD:C_0603_1608Metric_Pad1.08x0.95mm_HandSolder" H 6738 4150 50  0001 C CNN
+F 2 "Capacitor_SMD:C_1206_3216Metric_Pad1.33x1.80mm_HandSolder" H 6738 4150 50  0001 C CNN
 F 3 "" H 6700 4300 50  0001 C CNN
 	1    6700 4300
