File: msi2500.sch (KiCad schematic (older format))
At the start: 29 parts, among them J1 VCC_GPIO, J2 GPIO0, J3 GPIO1, J4 GPIO2, J5 GPIO3, U1 msi2500, Y1 24MHz, Y2 24MHZ

Commit message: Changed the package of R, C and L to 1206 for hand soldering.
Parts:
- C1, C10, C42, C9: footprint Capacitors_SMD:C_0603 -> Capacitor_SMD:C_1206_3216Metric_Pad1.33x1.80mm_HandSolder
- C2, C3, C39, C4, C41, C5, C6, C7, C8: footprint Capacitors_SMD:C_0805 -> Capacitor_SMD:C_1206_3216Metric_Pad1.33x1.80mm_HandSolder
- D5: footprint Diodes_THT:D_DO-35_SOD27_P2.54mm_Vertical_AnodeUp -> Diode_THT:D_DO-35_SOD27_P2.54mm_Vertical_AnodeUp
- J1, J2, J3, J4, J5: footprint Connectors:Pin_d0.7mm_L6.5mm_W1.8mm_FlatFork -> Connector_Pin:Pin_D0.7mm_L6.5mm_W1.8mm_FlatFork
- R1, R3, R4, R5, R6, R7, R8: footprint Resistors_SMD:R_0603 -> Resistor_SMD:R_1206_3216Metric_Pad1.30x1.75mm_HandSolder
- U1: footprint Housings_DFN_QFN:QFN-32-1EP_5x5mm_Pitch0.5mm -> Package_DFN_QFN:QFN-32-1EP_5x5mm_P0.5mm_EP3.7x3.7mm_ThermalVias
- Y1: footprint Crystals:Crystal_HC50_Vertical -> Crystal:Crystal_HC50_Vertical
- Y2: footprint Crystals:Crystal_SMD_7050-4pin_7.0x5.0mm -> Crystal:Crystal_SMD_7050-4Pin_7.0x5.0mm
Changed lines of the file:
@@
 F 0 "C1" H 4075 4250 50  0000 L CNN
 F 1 "10nF" H 4075 4050 50  0000 L CNN
-F 2 "Capacitors_SMD:C_0603" H 4088 4000 50  0001 C CNN
+F 2 "Capacitor_SMD:C_1206_3216Metric_Pad1.33x1.80mm_HandSolder" H 4088 4000 50  0001 C CNN
 F 3 "" H 4050 4150 50  0001 C CNN
 	1    4050 4150
@@
 F 0 "C4" H 4875 5600 50  0000 L CNN
 F 1 "10uF" H 4875 5400 50  0000 L CNN
-F 2 "Capacitors_SMD:C_0805" H 4888 5350 50  0001 C CNN
+F 2 "Capacitor_SMD:C_1206_3216Metric_Pad1.33x1.80mm_HandSolder" H 4888 5350 50  0001 C CNN
 F 3 "" H 4850 5500 50  0001 C CNN
 	1    4850 5500
@@
 F 0 "C8" H 6975 5550 50  0000 L CNN
 F 1 "1uF" H 6975 5350 50  0000 L CNN
-F 2 "Capacitors_SMD:C_0805" H 6988 5300 50  0001 C CNN
+F 2 "Capacitor_SMD:C_1206_3216Metric_Pad1.33x1.80mm_HandSolder" H 6988 5300 50  0001 C CNN
 F 3 "" H 6950 5450 50  0001 C CNN
 	1    6950 5450
@@
 F 0 "C5" H 5525 6000 50  0000 L CNN
 F 1 "10uF" H 5525 5800 50  0000 L CNN
-F 2 "Capacitors_SMD:C_0805" H 5538 5750 50  0001 C CNN
+F 2 "Capacitor_SMD:C_1206_3216Metric_Pad1.33x1.80mm_HandSolder" H 5538 5750 50  0001 C CNN
 F 3 "" H 5500 5900 50  0001 C CNN
 	1    5500 5900
@@
 F 0 "C6" H 5825 6000 50  0000 L CNN
 F 1 "1uF" H 5825 5800 50  0000 L CNN
-F 2 "Capacitors_SMD:C_0805" H 5838 5750 50  0001 C CNN
+F 2 "Capacitor_SMD:C_1206_3216Metric_Pad1.33x1.80mm_HandSolder" H 5838 5750 50  0001 C CNN
 F 3 "" H 5800 5900 50  0001 C CNN
 	1    5800 5900
@@
 F 0 "R1" V 6980 3800 50  0000 C CNN
 F 1 "510R" V 6900 3800 50  0000 C CNN
-F 2 "Resistors_SMD:R_0603" V 6830 3800 50  0001 C CNN
+F 2 "Resistor_SMD:R_1206_3216Metric_Pad1.30x1.75mm_HandSolder" V 6830 3800 50  0001 C CNN
 F 3 "" H 6900 3800 50  0001 C CNN
 	1    6900 3800
@@
 F 0 "Y1" H 7100 3550 50  0000 C CNN
 F 1 "24MHz" H 7100 3250 50  0000 C CNN
-F 2 "Crystals:Crystal_HC50_Vertical" H 7100 3400 50  0001 C CNN
+F 2 "Crystal:Crystal_HC50_Vertical" H 7100 3400 50  0001 C CNN
 F 3 "" H 7100 3400 50  0001 C CNN
 	1    7100 3400
@@
 F 0 "C9" H 7525 3300 50  0000 L CNN
 F 1 "18pF" H 7300 3100 50  0000 L CNN
-F 2 "Capacitors_SMD:C_0603" H 7538 3050 50  0001 C CNN
+F 2 "Capacitor_SMD:C_1206_3216Metric_Pad1.33x1.80mm_HandSolder" H 7538 3050 50  0001 C CNN
 F 3 "" H 7500 3200 50  0001 C CNN
 	1    7500 3200
@@
 F 0 "C10" H 7525 3700 50  0000 L CNN
 F 1 "18pF" H 7300 3500 50  0000 L CNN
-F 2 "Capacitors_SMD:C_0603" H 7538 3450 50  0001 C CNN
+F 2 "Capacitor_SMD:C_1206_3216Metric_Pad1.33x1.80mm_HandSolder" H 7538 3450 50  0001 C CNN
 F 3 "" H 7500 3600 50  0001 C CNN
 	1    7500 3600
@@
 F 0 "C3" H 4775 2900 50  0000 L CNN
 F 1 "10uF" H 4775 2700 50  0000 L CNN
-F 2 "Capacitors_SMD:C_0805" H 4788 2650 50  0001 C CNN
+F 2 "Capacitor_SMD:C_1206_3216Metric_Pad1.33x1.80mm_HandSolder" H 4788 2650 50  0001 C CNN
 F 3 "" H 4750 2800 50  0001 C CNN
 	1    4750 2800
@@
 F 0 "C2" H 4775 2150 50  0000 L CNN
 F 1 "10uF" H 4775 1950 50  0000 L CNN
-F 2 "Capacitors_SMD:C_0805" H 4788 1900 50  0001 C CNN
+F 2 "Capacitor_SMD:C_1206_3216Metric_Pad1.33x1.80mm_HandSolder" H 4788 1900 50  0001 C CNN
 F 3 "" H 4750 2050 50  0001 C CNN
 	1    4750 2050
@@
 F 0 "C7" H 6825 4500 50  0000 L CNN
 F 1 "10uF" H 6825 4300 50  0000 L CNN
-F 2 "Capacitors_SMD:C_0805" H 6838 4250 50  0001 C CNN
+F 2 "Capacitor_SMD:C_1206_3216Metric_Pad1.33x1.80mm_HandSolder" H 6838 4250 50  0001 C CNN
 F 3 "" H 6800 4400 50  0001 C CNN
 	1    6800 4400
@@
 F 0 "U1" H 4900 3400 60  0000 C CNN
 F 1 "msi2500" H 5500 2900 60  0000 C CNN
-F 2 "Housings_DFN_QFN:QFN-32-1EP_5x5mm_Pitch0.5mm" H 4900 3400 60  0001 C CNN
+F 2 "Package_DFN_QFN:QFN-32-1EP_5x5mm_P0.5mm_EP3.7x3.7mm_ThermalVias" H 4900 3400 60  0001 C CNN
 F 3 "" H 4900 3400 60  0001 C CNN
 	1    4900 3400
@@
 F 0 "J1" H 3500 3100 50  0000 C CNN
 F 1 "VCC_GPIO" H 3500 2900 50  0000 C CNN
-F 2 "Connectors:Pin_d0.7mm_L6.5mm_W1.8mm_FlatFork" H 3500 3000 50  0001 C CNN
+F 2 "Connector_Pin:Pin_D0.7mm_L6.5mm_W1.8mm_FlatFork" H 3500 3000 50  0001 C CNN
 F 3 "" H 3500 3000 50  0001 C CNN
 	1    3500 3000
@@
 F 0 "J2" H 3500 3400 50  0000 C CNN
 F 1 "GPIO0" H 3500 3200 50  0000 C CNN
-F 2 "Connectors:Pin_d0.7mm_L6.5mm_W1.8mm_FlatFork" H 3500 3300 50  0001 C CNN
+F 2 "Connector_Pin:Pin_D0.7mm_L6.5mm_W1.8mm_FlatFork" H 3500 3300 50  0001 C CNN
 F 3 "" H 3500 3300 50  0001 C CNN
 	1    3500 3300
@@
 F 0 "J3" H 3500 3700 50  0000 C CNN
 F 1 "GPIO1" H 3500 3500 50  0000 C CNN
-F 2 "Connectors:Pin_d0.7mm_L6.5mm_W1.8mm_FlatFork" H 3500 3600 50  0001 C CNN
+F 2 "Connector_Pin:Pin_D0.7mm_L6.5mm_W1.8mm_FlatFork" H 3500 3600 50  0001 C CNN
 F 3 "" H 3500 3600 50  0001 C CNN
 	1    3500 3600
@@
 F 0 "J4" H 3500 4000 50  0000 C CNN
 F 1 "GPIO2" H 3500 3800 50  0000 C CNN
-F 2 "Connectors:Pin_d0.7mm_L6.5mm_W1.8mm_FlatFork" H 3500 3900 50  0001 C CNN
+F 2 "Connector_Pin:Pin_D0.7mm_L6.5mm_W1.8mm_FlatFork" H 3500 3900 50  0001 C CNN
 F 3 "" H 3500 3900 50  0001 C CNN
 	1    3500 3900
@@
 F 0 "J5" H 3500 4300 50  0000 C CNN
 F 1 "GPIO3" H 3500 4100 50  0000 C CNN
-F 2 "Connectors:Pin_d0.7mm_L6.5mm_W1.8mm_FlatFork" H 3500 4200 50  0001 C CNN
+F 2 "Connector_Pin:Pin_D0.7mm_L6.5mm_W1.8mm_FlatFork" H 3500 4200 50  0001 C CNN
 F 3 "" H 3500 4200 50  0001 C CNN
 	1    3500 4200
@@
 F 0 "C39" H 6525 4550 50  0000 L CNN
 F 1 "1UF" H 6525 4350 50  0000 L CNN
-F 2 "Capacitors_SMD:C_0805" H 6538 4300 50  0001 C CNN
+F 2 "Capacitor_SMD:C_1206_3216Metric_Pad1.33x1.80mm_HandSolder" H 6538 4300 50  0001 C CNN
 F 3 "" H 6500 4450 50  0001 C CNN
 	1    6500 4450
@@
 F 0 "Y2" V 7350 2750 50  0000 L CNN
 F 1 "24MHZ" V 7500 2550 50  0000 L CNN
-F 2 "Crystals:Crystal_SMD_7050-4pin_7.0x5.0mm" H 7150 2450 50  0001 C CNN
+F 2 "Crystal:Crystal_SMD_7050-4Pin_7.0x5.0mm" H 7150 2450 50  0001 C CNN
 F 3 "" H 7150 2450 50  0001 C CNN
 	1    7150 2450
@@
 F 0 "D5" H 8800 4150 50  0000 C CNN
 F 1 "LED" H 8800 3950 50  0000 C CNN
-F 2 "Diodes_THT:D_DO-35_SOD27_P2.54mm_Vertical_AnodeUp" H 8800 4050 50  0001 C CNN
+F 2 "Diode_THT:D_DO-35_SOD27_P2.54mm_Vertical_AnodeUp" H 8800 4050 50  0001 C CNN
 F 3 "" H 8800 4050 50  0001 C CNN
 	1    8800 4050
@@
 F 0 "R3" V 8880 3500 50  0000 C CNN
 F 1 "512" V 8800 3500 50  0000 C CNN
-F 2 "Resistors_SMD:R_0603" V 8730 3500 50  0001 C CNN
+F 2 "Resistor_SMD:R_1206_3216Metric_Pad1.30x1.75mm_HandSolder" V 8730 3500 50  0001 C CNN
 F 3 "" H 8800 3500 50  0001 C CNN
 	1    8800 3500
@@
 F 0 "R4" V 6830 2600 50  0000 C CNN
 F 1 "10K" V 6750 2600 50  0000 C CNN
-F 2 "Resistors_SMD:R_0603" V 6680 2600 50  0001 C CNN
+F 2 "Resistor_SMD:R_1206_3216Metric_Pad1.30x1.75mm_HandSolder" V 6680 2600 50  0001 C CNN
 F 3 "" H 6750 2600 50  0001 C CNN
 	1    6750 2600
@@
 F 0 "R7" V 3230 4300 50  0000 C CNN
 F 1 "10K" V 3150 4300 50  0000 C CNN
-F 2 "Resistors_SMD:R_0603" V 3080 4300 50  0001 C CNN
+F 2 "Resistor_SMD:R_1206_3216Metric_Pad1.30x1.75mm_HandSolder" V 3080 4300 50  0001 C CNN
 F 3 "" H 3150 4300 50  0001 C CNN
 	1    3150 4300
@@
 F 0 "R6" V 3030 3900 50  0000 C CNN
 F 1 "10K" V 2950 3900 50  0000 C CNN
-F 2 "Resistors_SMD:R_0603" V 2880 3900 50  0001 C CNN
+F 2 "Resistor_SMD:R_1206_3216Metric_Pad1.30x1.75mm_HandSolder" V 2880 3900 50  0001 C CNN
 F 3 "" H 2950 3900 50  0001 C CNN
 	1    2950 3900
@@
 F 0 "R5" V 2830 3900 50  0000 C CNN
 F 1 "10K" V 2750 3900 50  0000 C CNN
-F 2 "Resistors_SMD:R_0603" V 2680 3900 50  0001 C CNN
+F 2 "Resistor_SMD:R_1206_3216Metric_Pad1.30x1.75mm_HandSolder" V 2680 3900 50  0001 C CNN
 F 3 "" H 2750 3900 50  0001 C CNN
 	1    2750 3900
@@
 F 0 "R8" V 3980 4400 50  0000 C CNN
 F 1 "10K" V 3900 4400 50  0000 C CNN
-F 2 "Resistors_SMD:R_0603" V 3830 4400 50  0001 C CNN
+F 2 "Resistor_SMD:R_1206_3216Metric_Pad1.30x1.75mm_HandSolder" V 3830 4400 50  0001 C CNN
 F 3 "" H 3900 4400 50  0001 C CNN
 	1    3900 4400
@@
 F 0 "C41" H 3875 2750 50  0000 L CNN
 F 1 "1UF" H 3875 2550 50  0000 L CNN
-F 2 "Capacitors_SMD:C_0805" H 3888 2500 50  0001 C CNN
+F 2 "Capacitor_SMD:C_1206_3216Metric_Pad1.33x1.80mm_HandSolder" H 3888 2500 50  0001 C CNN
 F 3 "" H 3850 2650 50  0001 C CNN
 	1    3850 2650
@@
 F 0 "C42" H 6375 3450 50  0000 L CNN
 F 1 "10nF" H 6375 3250 50  0000 L CNN
-F 2 "Capacitors_SMD:C_0603" H 6388 3200 50  0001 C CNN
+F 2 "Capacitor_SMD:C_1206_3216Metric_Pad1.33x1.80mm_HandSolder" H 6388 3200 50  0001 C CNN
 F 3 "" H 6350 3350 50  0001 C CNN
 	1    6350 3350
