File: rf_parts.sch (KiCad schematic (older format))
At the start: 20 parts, among them J10 SMA_VHF1, J12 Conn_01x02, J6 SMA_0_30MHZ, J7 SMA_30_60MHZ, J8 SMA_VHF2, J9 SMA_UHF

Commit message: Changed the package of R, C and L to 1206 for hand soldering.
Parts:
- C27: footprint Capacitors_SMD:C_0805 -> Capacitor_SMD:C_1206_3216Metric_Pad1.33x1.80mm_HandSolder
- C28, C29, C30, C31, C32, C33, C34: footprint Capacitors_SMD:C_0603 -> Capacitor_SMD:C_1206_3216Metric_Pad1.33x1.80mm_HandSolder
- J10, J8, J9: footprint sma:SMA_OPL_EMPTYHEAD -> Connector_Coaxial:SMA_Samtec_SMA-J-P-X-ST-EM1_EdgeMount
- J6, J7: footprint sma:SMA_OPL_EM -> Connector_Coaxial:SMA_Samtec_SMA-J-P-X-ST-EM1_EdgeMount
- L1, L2, L3, L4, L5, L6: footprint Inductors_SMD:L_0805 -> Inductor_SMD:L_1206_3216Metric_Pad1.42x1.75mm_HandSolder
Changed lines of the file:
@@
 F 0 "L3" V 3950 2500 50  0000 C CNN
 F 1 "330nH" V 4075 2500 50  0000 C CNN
-F 2 "Inductors_SMD:L_0805" H 4000 2500 50  0001 C CNN
+F 2 "Inductor_SMD:L_1206_3216Metric_Pad1.42x1.75mm_HandSolder" H 4000 2500 50  0001 C CNN
 F 3 "" H 4000 2500 50  0001 C CNN
 	1    4000 2500
@@
 F 0 "C27" H 3275 2600 50  0000 L CNN
 F 1 "470nF" H 3275 2400 50  0000 L CNN
-F 2 "Capacitors_SMD:C_0805" H 3288 2350 50  0001 C CNN
+F 2 "Capacitor_SMD:C_1206_3216Metric_Pad1.33x1.80mm_HandSolder" H 3288 2350 50  0001 C CNN
 F 3 "" H 3250 2500 50  0001 C CNN
 	1    3250 2500
@@
 F 0 "C29" H 3775 3300 50  0000 L CNN
 F 1 "56pF" H 3775 3100 50  0000 L CNN
-F 2 "Capacitors_SMD:C_0603" H 3788 3050 50  0001 C CNN
+F 2 "Capacitor_SMD:C_1206_3216Metric_Pad1.33x1.80mm_HandSolder" H 3788 3050 50  0001 C CNN
 F 3 "" H 3750 3200 50  0001 C CNN
 	1    3750 3200
@@
 F 0 "L1" V 2800 4250 50  0000 C CNN
 F 1 "220nH" V 2925 4250 50  0000 C CNN
-F 2 "Inductors_SMD:L_0805" H 2850 4250 50  0001 C CNN
+F 2 "Inductor_SMD:L_1206_3216Metric_Pad1.42x1.75mm_HandSolder" H 2850 4250 50  0001 C CNN
 F 3 "" H 2850 4250 50  0001 C CNN
 	1    2850 4250
@@
 F 0 "C30" H 3875 4350 50  0000 L CNN
 F 1 "3.9pF" H 3875 4150 50  0000 L CNN
-F 2 "Capacitors_SMD:C_0603" H 3888 4100 50  0001 C CNN
+F 2 "Capacitor_SMD:C_1206_3216Metric_Pad1.33x1.80mm_HandSolder" H 3888 4100 50  0001 C CNN
 F 3 "" H 3850 4250 50  0001 C CNN
 	1    3850 4250
@@
 F 0 "L2" V 3800 4650 50  0000 C CNN
 F 1 "330nH" V 3925 4650 50  0000 C CNN
-F 2 "Inductors_SMD:L_0805" H 3850 4650 50  0001 C CNN
+F 2 "Inductor_SMD:L_1206_3216Metric_Pad1.42x1.75mm_HandSolder" H 3850 4650 50  0001 C CNN
 F 3 "" H 3850 4650 50  0001 C CNN
 	1    3850 4650
@@
 F 0 "C32" H 4925 4500 50  0000 L CNN
 F 1 "39pF" H 4925 4300 50  0000 L CNN
-F 2 "Capacitors_SMD:C_0603" H 4938 4250 50  0001 C CNN
+F 2 "Capacitor_SMD:C_1206_3216Metric_Pad1.33x1.80mm_HandSolder" H 4938 4250 50  0001 C CNN
 F 3 "" H 4900 4400 50  0001 C CNN
 	1    4900 4400
@@
 F 0 "C28" H 3275 3050 50  0000 L CNN
 F 1 "1nF" H 3275 2850 50  0000 L CNN
-F 2 "Capacitors_SMD:C_0603" H 3288 2800 50  0001 C CNN
+F 2 "Capacitor_SMD:C_1206_3216Metric_Pad1.33x1.80mm_HandSolder" H 3288 2800 50  0001 C CNN
 F 3 "" H 3250 2950 50  0001 C CNN
 	1    3250 2950
@@
 F 0 "L4" V 4400 2500 50  0000 C CNN
 F 1 "270nH" V 4525 2500 50  0000 C CNN
-F 2 "Inductors_SMD:L_0805" H 4450 2500 50  0001 C CNN
+F 2 "Inductor_SMD:L_1206_3216Metric_Pad1.42x1.75mm_HandSolder" H 4450 2500 50  0001 C CNN
 F 3 "" H 4450 2500 50  0001 C CNN
 	1    4450 2500
@@
 F 0 "L5" V 4850 2500 50  0000 C CNN
 F 1 "150nH" V 4975 2500 50  0000 C CNN
-F 2 "Inductors_SMD:L_0805" H 4900 2500 50  0001 C CNN
+F 2 "Inductor_SMD:L_1206_3216Metric_Pad1.42x1.75mm_HandSolder" H 4900 2500 50  0001 C CNN
 F 3 "" H 4900 2500 50  0001 C CNN
 	1    4900 2500
@@
 F 0 "L6" V 5300 2500 50  0000 C CNN
 F 1 "330nH" V 5425 2500 50  0000 C CNN
-F 2 "Inductors_SMD:L_0805" H 5350 2500 50  0001 C CNN
+F 2 "Inductor_SMD:L_1206_3216Metric_Pad1.42x1.75mm_HandSolder" H 5350 2500 50  0001 C CNN
 F 3 "" H 5350 2500 50  0001 C CNN
 	1    5350 2500
@@
 F 0 "C31" H 4275 3300 50  0000 L CNN
 F 1 "160pF" H 4275 3100 50  0000 L CNN
-F 2 "Capacitors_SMD:C_0603" H 4288 3050 50  0001 C CNN
+F 2 "Capacitor_SMD:C_1206_3216Metric_Pad1.33x1.80mm_HandSolder" H 4288 3050 50  0001 C CNN
 F 3 "" H 4250 3200 50  0001 C CNN
 	1    4250 3200
@@
 F 0 "C33" H 5175 3300 50  0000 L CNN
 F 1 "160pF" H 5175 3100 50  0000 L CNN
-F 2 "Capacitors_SMD:C_0603" H 5188 3050 50  0001 C CNN
+F 2 "Capacitor_SMD:C_1206_3216Metric_Pad1.33x1.80mm_HandSolder" H 5188 3050 50  0001 C CNN
 F 3 "" H 5150 3200 50  0001 C CNN
 	1    5150 3200
@@
 F 0 "C34" H 5775 3300 50  0000 L CNN
 F 1 "56pF" H 5775 3100 50  0000 L CNN
-F 2 "Capacitors_SMD:C_0603" H 5788 3050 50  0001 C CNN
+F 2 "Capacitor_SMD:C_1206_3216Metric_Pad1.33x1.80mm_HandSolder" H 5788 3050 50  0001 C CNN
 F 3 "" H 5750 3200 50  0001 C CNN
 	1    5750 3200
@@
 F 0 "J6" H 1800 2800 50  0000 C CNN
 F 1 "SMA_0_30MHZ" H 1800 2400 50  0000 C CNN
-F 2 "sma:SMA_OPL_EM" H 1800 2600 50  0001 C CNN
+F 2 "Connector_Coaxial:SMA_Samtec_SMA-J-P-X-ST-EM1_EdgeMount" H 1800 2600 50  0001 C CNN
 F 3 "" H 1800 2600 50  0001 C CNN
 	1    1800 2600
@@
 F 0 "J7" H 1900 4550 50  0000 C CNN
 F 1 "SMA_30_60MHZ" H 1900 4150 50  0000 C CNN
-F 2 "sma:SMA_OPL_EM" H 1900 4350 50  0001 C CNN
+F 2 "Connector_Coaxial:SMA_Samtec_SMA-J-P-X-ST-EM1_EdgeMount" H 1900 4350 50  0001 C CNN
 F 3 "" H 1900 4350 50  0001 C CNN
 	1    1900 4350
@@
 F 0 "J8" H 8150 3000 50  0000 C CNN
 F 1 "SMA_VHF2" H 8150 2600 50  0000 C CNN
-F 2 "sma:SMA_OPL_EMPTYHEAD" H 8150 2800 50  0001 C CNN
+F 2 "Connector_Coaxial:SMA_Samtec_SMA-J-P-X-ST-EM1_EdgeMount" H 8150 2800 50  0001 C CNN
 F 3 "" H 8150 2800 50  0001 C CNN
 	1    8150 2800
@@
 F 0 "J9" H 8150 3750 50  0000 C CNN
 F 1 "SMA_UHF" H 8150 3350 50  0000 C CNN
-F 2 "sma:SMA_OPL_EMPTYHEAD" H 8150 3550 50  0001 C CNN
+F 2 "Connector_Coaxial:SMA_Samtec_SMA-J-P-X-ST-EM1_EdgeMount" H 8150 3550 50  0001 C CNN
 F 3 "" H 8150 3550 50  0001 C CNN
 	1    8150 3550
@@
 F 0 "J10" H 8150 4500 50  0000 C CNN
 F 1 "SMA_VHF1" H 8150 4100 50  0000 C CNN
-F 2 "sma:SMA_OPL_EMPTYHEAD" H 8150 4300 50  0001 C CNN
+F 2 "Connector_Coaxial:SMA_Samtec_SMA-J-P-X-ST-EM1_EdgeMount" H 8150 4300 50  0001 C CNN
 F 3 "" H 8150 4300 50  0001 C CNN
 	1    8150 4300
